File: xmit/_autosave-xmit.kicad_pcb (KiCad board)
At the start: 4 copper layers, 59.8 x 36.7 mm, 31 parts, among them U1 74LVC1G66, U2 74LVC1G66, U3 74LVC1G66, U4 74LVC1G66, U5 74LVC1G66, U6 74LVC1G66

Commit message: First round WIP on the filters and amplifier
Parts:
- moved C10 4.06 mm to (180.8, 79.9)
- moved L4 3.51 mm to (180.8, 83.0)
- moved U3 1.80 mm to (159.2, 81.5)
Routing:
- net /transmit filters/band_30: track 0.00 -> 36.7 mm, vias 0 -> 2
- net /transmit filters/band_20: track 0.00 -> 35.7 mm, vias 0 -> 2
- net /transmit filters/band_10: track 0.00 -> 35.6 mm, vias 0 -> 2
- net Net-(U7-D1_IN+): track 9.97 -> 30.0 mm
- net GND: track 20.3 -> 30.4 mm, vias 14 -> 19
- net Net-(C4-Pad1): track 9.08 -> 18.4 mm
- net Net-(C14-Pad1): track 7.71 -> 16.9 mm
- net Net-(C3-Pad1): track 7.68 -> 16.3 mm
- net Net-(U7-D2_IN+): track 0.00 -> 4.66 mm, vias 0 -> 2
- net Net-(C5-Pad2): track 13.7 -> 14.5 mm
- net Net-(C10-Pad2): track 14.7 -> 14.2 mm
