File: xmit/rf-power.kicad_sch (KiCad schematic)
At the start: 9 parts

Commit message: More layout cleanup.
This is a checkpoint before I move all of the power management to a separate board. Next step is to move all power management to a separate board.
Parts:
- renumbered C24 to C401, C25 to C402, R41 to R401, R42 to R402, R46 to R403, R43 to R404, R44 to R405, R45 to R406, U8 to U401
Changed lines of the file:
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@@
 		(in_pos_files yes)
 		(dnp no)
-		(property "Reference" "#PWR037"
+		(property "Reference" "#PWR0401"
 			(at 120.65 100.33 0)
 			(hide yes)
@@
 			(project "xmit"
 				(path "/938afe95-c1c4-4cca-88b7-71a9df9e4417/0c0ed751-8a03-405a-972d-dcacaa180c8b"
-					(reference "#PWR037")
+					(reference "#PWR0401")
 					(unit 1)
 				)
@@
 		(in_pos_files yes)
 		(dnp no)
-		(property "Reference" "#PWR039"
+		(property "Reference" "#PWR0403"
 			(at 139.7 109.22 0)
 			(hide yes)
@@
 			(project "xmit"
 				(path "/938afe95-c1c4-4cca-88b7-71a9df9e4417/0c0ed751-8a03-405a-972d-dcacaa180c8b"
-					(reference "#PWR039")
+					(reference "#PWR0403")
 					(unit 1)
 				)
@@
 		(in_pos_files yes)
 		(dnp no)
-		(property "Reference" "C25"
+		(property "Reference" "C402"
 			(at 113.03 88.392 0)
 			(show_name no)
@@
 			(project "xmit"
 				(path "/938afe95-c1c4-4cca-88b7-71a9df9e4417/0c0ed751-8a03-405a-972d-dcacaa180c8b"
-					(reference "C25")
+					(reference "C402")
 					(unit 1)
 				)
@@
 		(dnp no)
 		(fields_autoplaced yes)
-		(property "Reference" "R42"
+		(property "Reference" "R402"
 			(at 173.99 73.6599 0)
 			(show_name no)
@@
 			(project "xmit"
 				(path "/938afe95-c1c4-4cca-88b7-71a9df9e4417/0c0ed751-8a03-405a-972d-dcacaa180c8b"
-					(reference "R42")
+					(reference "R402")
 					(unit 1)
 				)
@@
 		(dnp no)
 		(fields_autoplaced yes)
-		(property "Reference" "R43"
+		(property "Reference" "R404"
 			(at 173.99 93.9799 0)
 			(show_name no)
@@
 			(project "xmit"
 				(path "/938afe95-c1c4-4cca-88b7-71a9df9e4417/0c0ed751-8a03-405a-972d-dcacaa180c8b"
-					(reference "R43")
+					(reference "R404")
 					(unit 1)
 				)
@@
 		(in_pos_files yes)
 		(dnp no)
-		(property "Reference" "R45"
+		(property "Reference" "R406"
 			(at 186.69 98.044 90)
 			(show_name no)
@@
 			(project "xmit"
 				(path "/938afe95-c1c4-4cca-88b7-71a9df9e4417/0c0ed751-8a03-405a-972d-dcacaa180c8b"
-					(reference "R45")
+					(reference "R406")
 					(unit 1)
 				)
@@
 		(dnp no)
 		(fields_autoplaced yes)
-		(property "Reference" "#PWR027"
+		(property "Reference" "#PWR0404"
 			(at 148.59 66.04 0)
 			(hide yes)
@@
 			(project "xmit"
 				(path "/938afe95-c1c4-4cca-88b7-71a9df9e4417/0c0ed751-8a03-405a-972d-dcacaa180c8b"
-					(reference "#PWR027")
+					(reference "#PWR0404")
 					(unit 1)
 				)
@@
 		(dnp no)
 		(fields_autoplaced yes)
-		(property "Reference" "R46"
+		(property "Reference" "R403"
 			(at 173.99 83.8199 0)
 			(show_name no)
@@
 			(project "xmit"
 				(path "/938afe95-c1c4-4cca-88b7-71a9df9e4417/0c0ed751-8a03-405a-972d-dcacaa180c8b"
-					(reference "R46")
+					(reference "R403")
 					(unit 1)
 				)
@@
 		(in_pos_files yes)
 		(dnp no)
-		(property "Reference" "U8"
+		(property "Reference" "U401"
 			(at 143.51 86.106 0)
 			(show_name no)
@@
 			)
 		)
-		(property "Datasheet" ""
+		(property "Datasheet" "https://www.ti.com/lit/ds/symlink/ths6222.pdf"
 			(at 144.78 85.09 0)
 			(hide yes)
@@
 			(project "xmit"
 				(path "/938afe95-c1c4-4cca-88b7-71a9df9e4417/0c0ed751-8a03-405a-972d-dcacaa180c8b"
-					(reference "U8")
+					(reference "U401")
 					(unit 1)
 				)
@@
 		(dnp no)
 		(fields_autoplaced yes)
-		(property "Reference" "C24"
+		(property "Reference" "C401"
 			(at 118.11 58.42 90)
 			(show_name no)
@@
 			(project "xmit"
 				(path "/938afe95-c1c4-4cca-88b7-71a9df9e4417/0c0ed751-8a03-405a-972d-dcacaa180c8b"
-					(reference "C24")
+					(reference "C401")
 					(unit 1)
 				)
@@
 		(in_pos_files yes)
 		(dnp no)
-		(property "Reference" "R41"
+		(property "Reference" "R401"
 			(at 168.148 63.754 90)
 			(show_name no)
@@
 			(project "xmit"
 				(path "/938afe95-c1c4-4cca-88b7-71a9df9e4417/0c0ed751-8a03-405a-972d-dcacaa180c8b"
-					(reference "R41")
+					(reference "R401")
 					(unit 1)
 				)
@@
 		(in_pos_files yes)
 		(dnp no)
-		(property "Reference" "R44"
+		(property "Reference" "R405"
 			(at 186.69 67.564 90)
 			(show_name no)
@@
 			(project "xmit"
 				(path "/938afe95-c1c4-4cca-88b7-71a9df9e4417/0c0ed751-8a03-405a-972d-dcacaa180c8b"
-					(reference "R44")
+					(reference "R405")
 					(unit 1)
 				)
@@
 		(in_pos_files yes)
 		(dnp no)
-		(property "Reference" "#PWR040"
+		(property "Reference" "#PWR0402"
 			(at 137.16 68.58 0)
 			(hide yes)
@@
 			(project "xmit"
 				(path "/938afe95-c1c4-4cca-88b7-71a9df9e4417/0c0ed751-8a03-405a-972d-dcacaa180c8b"
-					(reference "#PWR040")
-					(unit 1)
-				)
+					(reference "#PWR0402")
+					(unit 1)
+				)

Commit message: changes up to first spin
Parts:
- C401, C402: value 100n -> 10n; KiLib_Generator (none) -> SMD_2terminal_chip_molded; LCSC Part # (none) -> C76626; now left out of the parts list
- R401, R402, R404: KiLib_Generator (none) -> SMD_2terminal_chip_molded; LCSC Part # (none) -> C852604
- R403: value 237 -> 240; KiLib_Generator (none) -> SMD_2terminal_chip_molded; LCSC (none) -> C102913; LCSC Part # (none) -> C17572
- R405, R406: value 2.5 -> 2; KiLib_Generator (none) -> SMD_2terminal_chip_molded; LCSC Part # (none) -> C101983; now left out of the parts list
- U401: value (none) -> THS6222IRHFR; KiLib_Generator (none) -> package/no_lead; LCSC Part # (none) -> C1855812
Connections:
- net +12V renamed +15V
