File: xmit/filter.kicad_sch (KiCad schematic)
At the start: 39 parts, among them U1 74LVC1G66, U11 SN74LVC1G04DBV, U12 74LVC1G66, U13 74LVC1G66, U2 74LVC1G66, U3 74LVC1G66, U4 74LVC1G66, U5 74LVC1G66, U6 74LVC1G66

Commit message: More layout cleanup.
This is a checkpoint before I move all of the power management to a separate board. Next step is to move all power management to a separate board.
Parts:
- renumbered C14 to C201, C3 to C202, C13 to C203, C4 to C204, C15 to C205, C5 to C206, C19 to C207, C6 to C208, C16 to C209, C7 to C210, C20 to C211, C8 to C212, C17 to C213, C9 to C214, C21 to C215, C10 to C216, C18 to C217, C11 to C218, C22 to C219, C12 to C220, L5 to L201, L1 to L202, L8 to L203, L2 to L204, L6 to L205, L3 to L206, L9 to L207, L4 to L208, R1 to R201, R2 to R202, U11 to U201, U1 to U202, U2 to U203, U12 to U204, U3 to U205, U4 to U206, U5 to U207, U13 to U208, U6 to U209
Connections:
- net drive: now reaches U201.4, U202.1, U203.1, U204.1, U205.1

Commit message: changes up to first spin
Parts:
- added D201, D202, D203, D204: LED, LED_SMD:LED_0603_1608Metric, symbol Device:LED
- added R203, R204, R205, R206: 100, Resistor_SMD:R_0603_1608Metric, symbol Device:R
- C201: value 220p -> 560p; KiLib_Generator (none) -> SMD_2terminal_chip_molded; LCSC Part # (none) -> C107119; now left out of the parts list
- C202: value 120p -> 270p; KiLib_Generator (none) -> SMD_2terminal_chip_molded; LCSC Part # (none) -> C107106; now left out of the parts list
- C203: value 50p -> 270p; KiLib_Generator (none) -> SMD_2terminal_chip_molded; LCSC Part # (none) -> C113828; now left out of the parts list
- C204: KiLib_Generator (none) -> SMD_2terminal_chip_molded; LCSC Part # (none) -> C107115; now left out of the parts list
- C205: value 12p -> 33p; KiLib_Generator (none) -> SMD_2terminal_chip_molded; LCSC Part # (none) -> C85970; now left out of the parts list
- C206: value 8.1p -> 18p; KiLib_Generator (none) -> SMD_2terminal_chip_molded; LCSC Part # (none) -> C113825; now left out of the parts list
- C207: value 3.9p -> 15p; KiLib_Generator (none) -> SMD_2terminal_chip_molded; LCSC Part # (none) -> C107110; now left out of the parts list
- C208: KiLib_Generator (none) -> SMD_2terminal_chip_molded; LCSC Part # (none) -> C519933
- C209: value 330p -> 820p; KiLib_Generator (none) -> SMD_2terminal_chip_molded; LCSC Part # (none) -> C309484; now left out of the parts list
- C210: value 200p -> 430p; KiLib_Generator (none) -> SMD_2terminal_chip_molded; LCSC Part # (none) -> C520006; now left out of the parts list
- C211: value 81p -> 430p; KiLib_Generator (none) -> SMD_2terminal_chip_molded; LCSC Part # (none) -> C126556; now left out of the parts list
- C212: value 72p -> 39p; KiLib_Generator (none) -> SMD_2terminal_chip_molded; LCSC Part # (none) -> C107117; now left out of the parts list
- C213: value 31p -> 75pF; KiLib_Generator (none) -> SMD_2terminal_chip_molded; LCSC Part # (none) -> C113832; now left out of the parts list
- C214: value 18p -> 39p; KiLib_Generator (none) -> SMD_2terminal_chip_molded; LCSC Part # (none) -> C76645; now left out of the parts list
- C215: value 9p -> 33p; KiLib_Generator (none) -> SMD_2terminal_chip_molded; LCSC Part # (none) -> C85970; now left out of the parts list
- C216: value 5.6p -> 10n; KiLib_Generator (none) -> SMD_2terminal_chip_molded; LCSC Part # (none) -> C76626; now left out of the parts list
- C217: value 220p -> 560p; KiLib_Generator (none) -> SMD_2terminal_chip_molded; LCSC Part # (none) -> C97881; now left out of the parts list
- C218: value 120p -> 270p; KiLib_Generator (none) -> SMD_2terminal_chip_molded; LCSC Part # (none) -> C2986280; now left out of the parts list
- C219: value 50p -> 270p; KiLib_Generator (none) -> SMD_2terminal_chip_molded; LCSC Part # (none) -> C2986280; now left out of the parts list
- C220: KiLib_Generator (none) -> SMD_2terminal_chip_molded; LCSC Part # (none) -> C85970; now left out of the parts list
- L201: value 2200n -> 810nH; KiLib_Generator (none) -> SMD_2terminal_chip_molded; LCSC Part # (none) -> C139231; now left out of the parts list
- L202, L206: value 1600n -> 810nH; KiLib_Generator (none) -> SMD_2terminal_chip_molded; LCSC Part # (none) -> C98996; now left out of the parts list
- L203, L207: value 800n -> 220nH; KiLib_Generator (none) -> SMD_2terminal_chip_molded; LCSC Part # (none) -> C108960; now left out of the parts list
- L204, L208: value 56n -> 56nH; KiLib_Generator (none) -> SMD_2terminal_chip_molded; LCSC Part # (none) -> C98996; now left out of the parts list
- L205: value 2000n -> 810nH; KiLib_Generator (none) -> SMD_2terminal_chip_molded; LCSC Part # (none) -> C98996; now left out of the parts list
- R201: KiLib_Generator (none) -> SMD_2terminal_chip_molded; LCSC Part # (none) -> C114567; now left out of the parts list
- R202: KiLib_Generator (none) -> SMD_2terminal_chip_molded; LCSC Part # (none) -> C17378; now left out of the parts list
- U201: footprint Package_TO_SOT_SMD:SOT-23-5_HandSoldering -> Package_TO_SOT_SMD:SOT-23-5; KiLib_Generator (none) -> package/gullwing; LCSC Part # (none) -> C45367201; now left out of the parts list
- U202, U203, U204, U205, U206, U207, U208, U209: footprint Package_TO_SOT_SMD:SOT-23-5_HandSoldering -> Package_TO_SOT_SMD:SOT-23-5; KiLib_Generator (none) -> package/gullwing; LCSC Part # (none) -> C113518
Connections:
- net GND: now also D201.1 (K), D202.1 (K), D203.1 (K), D204.1 (K)
- net band.10m: now also R205.1
- net band.20m: now also R204.2
- net band.2m: now also R206.1
- net band.30m: now also R203.1
- new net: D204.2 (A), R206.2
- new net: D203.2 (A), R205.2
- new net: D201.2 (A), R203.2
- new net: D202.2 (A), R204.1
