File: sim/filters.kicad_sch (KiCad schematic)
At the start: 68 parts

Commit message: changes up to first spin
Parts:
- added C42: 10n, symbol Device:C
- added C43, C47: 1n, symbol Device:C
- added C44: 68p, symbol Device:C
- added C45: 2.2n, symbol Device:C
- added C46: 150p, symbol Device:C
- added L12, L13: 820n, symbol Device:L
- added R52: 150, symbol Device:R
- added R53: 10k, symbol Device:R
- added R54: 10, symbol Device:R
- added R55: 200, symbol Device:R
- C11, C3: value 290p -> 270p
Connections:
- net GND: now also C43.2, C45.2, C47.2, R53.2, R55.2
- net at R10.1, R11.1, R12.1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: now also R52.1
- new net: C42.2, C43.1, C44.1, L12.1
- new net: C44.2, C45.1, C46.1, L12.2, L13.1
- new net: C46.2, C47.1, L13.2, R54.1
- new net: C42.1, R52.2, R53.1
- new net out.40m: R54.2, R55.1
Other:
- note added: "7.0 - 7.125 MHz"
- moved on the sheet: C1, C10, C11, C12, C13, C14, C15, C16, C17, C18, C2, C27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
